File: production/ESP32_Simple_IoT.kicad_sch (KiCad schematic)
At the start: 23 parts, among them J1 USB_C, J2 LOAD, K1 SRD-05VDC-SL-C, Q1 BC817, SW1 BOOT, SW2 RESET, U1 ESP32-WROOM-32, U2 AMS1117-3.3, U3 CP2102N

Commit message: Complete PCB design: schematic wiring, routing, Gerbers, and manufacturing files
- Programmatic schematic wiring: 34 wire connections, 21 nets, 0 ERC errors
- PCB routing via Python script (route_pcb.py): 159 tracks, 78 vias, 0 shorts/unconnected
- Generated Gerber package for JLCPCB (11 files + ZIP)
- Corrected CPL coordinates to match actual footprint positions
- All 16 LCSC parts verified in stock
- Added PROJECT_STATUS.md agent handoff document
- DRC: 45 warnings (inherent to QFN-28/USB-C pad spacing), 0 functional issues

Co-Authored-By: Claude Opus 4.6 <noreply@anthropic.com>
Connections:
- net +5V: now also K1.2
- net GND: now also D3.2 (A), R3.1, R5.2, U1.26 (IO4)
- net at K1.3: no longer J2.2 (Pin_2)
- net at K1.4: now also J2.2 (Pin_2)
- net ESP_RX: no longer names the net of U1.34 (RXD0), U3.26 (TXD)
- net ESP_TX: no longer names the net of U1.35 (TXD0), U3.25 (RXD)
