File: handoff/manufacturing/ESP32_Simple_IoT.kicad_pcb (KiCad board)
At the start: 2 copper layers, 80 x 60 mm, 32 parts, among them J1 USB_C_Receptacle_GCT_USB4105-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, J2 PhoenixContact_MC_1,5_2-G-3.8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, K1 Relay_SPDT_SANYOU_SRD_Series_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, Q1 SOT-23, SW1 SW_SPST_TL3342, SW2 SW_SPST_TL3342, U1 ESP32-WROOM-32, U2 SOT-223-3_TabPin2, U3 QFN-28-1EP_5x5mm_P0.5mm_EP3.3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

Commit message: Rev 2: D1 at y=38, clears K1 relay and all B.Cu signal corridors
D1 flyback diode moved from (30,40) to (30,38). Avoids:
- K1 relay body (extends to ~y=42) — 4mm clearance
- ESP_TX B.Cu corridor at y=34
- ESP_RX B.Cu corridor at y=32
- ESP_EN B.Cu corridor at y=36

DRC: 0 unconnected, 40 violations (down from 41 baseline), 7 shorts
(all pre-existing J1 USB-C area — same as manufactured Rev 1.2).

Co-Authored-By: Claude Opus 4.6 <noreply@anthropic.com>
Parts:
- moved D1 4.00 mm to (30.0, 38.0)
Connections:
- U3 pad : (no net) -> GND
Routing:
- net RELAY_COIL: track 48.8 -> 46.9 mm
- net +5V: track 188.2 -> 189.7 mm
